File: Mk2/Mk2_PCB/hexapod_mk2_v0.0.brd (EAGLE design)
At the start: 80.5 x 61 mm, 16 parts

Commit message: Mk1 cleanup + PCB revisions
Parts:
- removed LEG6: 06-JST-B6B-XH-A, bt_con-jst-xh:B6B-XH
- added LED_RING: 03-JST-B3B-XH-A, bt_con-jst-xh:B3B-XH
- added LEG0: 06-JST-B6B-XH-A, bt_con-jst-xh:B6B-XH
- added R1: MPMT10014001AT1MPM_VIS, MPMT10014001AT1:MPM_VIS
- added S1: SWS004, smd-special:SMS-004
- added X1: JST-XH-02-PIN-LONG-PAD, Rembrandt Electronics - JST XH Connectors v1-0:JST-XH-02-PACKAGE-LONG-PAD
- 100R: value (none) -> 100
- 12V: value (none) -> Blue
- 470R: value (none) -> 470
- 5V: value (none) -> Red
- RPI5: value (none) -> Raspberry Pi
- moved LEG3 37.1 mm to (66.4, 3.40)
- moved LEG1 18.7 mm to (48.1, 40.5)
- moved LEG4 18.3 mm to (48.1, 3.40)
- moved LEG2 18.2 mm to (66.3, 40.5)
- moved LEG5 17.8 mm to (30.4, 3.40)
Connections:
- removed net 3V3: RPI5.1
- removed net 3V3_2: RPI5.17
- removed net GPIO10: RPI5.19
- removed net GPIO11: RPI5.23
- removed net GPIO12: RPI5.32
- removed net GPIO13: RPI5.33
- removed net GPIO16: RPI5.36
- removed net GPIO17: RPI5.11
- removed net GPIO18: RPI5.12
- removed net GPIO19: RPI5.35
- removed net GPIO2: RPI5.3
- removed net GPIO20: RPI5.38
- removed net GPIO21: RPI5.40
- removed net GPIO22: RPI5.15
- removed net GPIO23: RPI5.16
- removed net GPIO24: RPI5.18
- removed net GPIO25: RPI5.22
- removed net GPIO26: RPI5.37
- removed net GPIO27: RPI5.13
- removed net GPIO3: RPI5.5
- removed net GPIO4: RPI5.7
- removed net GPIO5: RPI5.29
- removed net GPIO6: RPI5.31
- removed net GPIO7: RPI5.26
- removed net GPIO8: RPI5.24
- removed net GPIO9: RPI5.21
- removed net ID_SC: RPI5.28
- removed net ID_SD: RPI5.27
- removed net L6M1: LEG6.P$3, U$1.19-A5/SCL0
- removed net L6M2: LEG6.P$4, U$1.22-A8/CTX1
- removed net L6M3: LEG6.P$5, U$1.23-A9/CRX1/MCLK1
- removed net L6SIG: LEG6.P$6, U$1.29-TX7
- new net 3.3V: RPI5.1, X1.1
- new net D_SW0: RPI5.22, S1.1
- new net D_SW1: RPI5.24, S1.2
- new net D_SW2: RPI5.26, S1.3
- new net D_SW3: RPI5.28, S1.4
- new net L0M1: LEG0.P$3, U$1.2-OUT2
- new net L0M2: LEG0.P$4, U$1.3-LRCLK2
- new net L0M3: LEG0.P$5, U$1.4-BCLK2
- new net L0SIG: LEG0.P$6, U$1.24-A10/TX6/SCL2
- new net LEDSIG: LED_RING.P$3, RPI5.33
- new net PWRSIG: RPI5.3, U$1.0-RX1/CS1/CRX2, X1.2
- new net V_DIV: R1.3, U$1.38-A14/CS/IN1
- net 12V: now also R1.1
- net 5V: now also LED_RING.P$1, LEG0.P$1, S1.5, S1.6, S1.7, S1.8; no longer LEG6.P$1
- net GND: now also LED_RING.P$2, LEG0.P$2, R1.2; no longer LEG6.P$2
- net L1M1: now also U$1.5-IN2; no longer U$1.2-OUT2
- net L1M2: now also U$1.6-OUT1D; no longer U$1.3-LRCLK2
- net L1M3: now also U$1.7-RX2/OUT1A; no longer U$1.4-BCLK2
- net L1SIG: now also U$1.25-A11/RX6/SDA2; no longer U$1.24-A10/TX6/SCL2
- net L2M1: now also U$1.8-TX2/IN2; no longer U$1.5-IN2
- net L2M2: now also U$1.9-OUT1C; no longer U$1.6-OUT1D
- net L2M3: now also U$1.10-CS\MQSR; no longer U$1.7-RX2/OUT1A
- net L2SIG: now also U$1.26-A12/MOSI1; no longer U$1.25-A11/RX6/SDA2
- net L3M1: now also U$1.11-MOSI/CTX1; no longer U$1.8-TX2/IN2
- net L3M2: now also U$1.12-MISO/MQSL; no longer U$1.9-OUT1C
- net L3M3: now also U$1.13-SCK/LED; no longer U$1.10-CS\MQSR
- net L3SIG: now also U$1.27-A13/SCK1; no longer U$1.26-A12/MOSI1
- net L4M1: now also U$1.14-A0/TX3/SPDIF_OUT; no longer U$1.11-MOSI/CTX1
- net L4M2: now also U$1.15-A1/RX3/SPDIF_IN; no longer U$1.12-MISO/MQSL
- net L4M3: now also U$1.18-A4/SDA0; no longer U$1.13-SCK/LED
- net L4SIG: now also U$1.28-RX7; no longer U$1.27-A13/SCK1
- net L5M1: now also U$1.19-A5/SCL0; no longer U$1.14-A0/TX3/SPDIF_OUT
- net L5M2: now also U$1.22-A8/CTX1; no longer U$1.15-A1/RX3/SPDIF_IN
- net L5M3: now also U$1.23-A9/CRX1/MCLK1; no longer U$1.18-A4/SDA0
- net L5SIG: now also U$1.29-TX7; no longer U$1.28-RX7
Routing:
- net L0M1: track 0.00 -> 57.4 mm
- net L6M2: track 53.2 -> 0.00 mm
- net L6M3: track 48.9 -> 0.00 mm
- net L0M2: track 0.00 -> 43.2 mm, vias 0 -> 1
- net L0M3: track 0.00 -> 43.2 mm, vias 0 -> 1
- net L6M1: track 36.2 -> 0.00 mm, vias 1 -> 0
- net L5M2: track 18.8 -> 53.2 mm
- net L6SIG: track 29.3 -> 0.00 mm
- net L5M3: track 22.8 -> 48.9 mm, vias 1 -> 0
- net L2SIG: track 11.1 -> 36.6 mm, vias 1 -> 0
- net L3M2: track 18.0 -> 42.8 mm
- net L3M3: track 16.9 -> 41.3 mm
- net L2M3: track 41.3 -> 16.9 mm
- net L4M2: track 42.8 -> 18.8 mm
- net L4M1: track 36.7 -> 13.8 mm
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
Commit message: Update Mk2 Schematic
Parts:
- added FAN: JST-XH-04-PIN-LONG-PAD, Rembrandt Electronics - JST XH Connectors v1-0:JST-XH-04-PACKAGE-LONG-PAD
Connections:
- new net FAN_PWM: FAN.1, RPI5.32
- new net FAN_RPM: FAN.2, RPI5.38
- net 12V: now also R1.2; no longer R1.1
- net 3.3V: now also S1.5, S1.6, S1.7, S1.8
- net 5V: now also FAN.3; no longer S1.5, S1.6, S1.7, S1.8
- net GND: now also FAN.4, R1.1; no longer R1.2
Changed lines of the file:
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@@
 <attribute name="VALUE" x="-19.8025" y="-39.1075" size="1.016" layer="27" ratio="10"/>
+</element>
+<element name="FAN" library="Rembrandt Electronics - JST XH Connectors v1-0" package="JST-XH-04-PACKAGE-LONG-PAD" value="JST-XH-04-PIN-LONG-PAD" x="-14" y="-51" smashed="yes">
+<attribute name="NAME" x="-20.655" y="-53.04" size="1.016" layer="25" ratio="10" rot="R90"/>
+<attribute name="VALUE" x="-20.0025" y="-47.1075" size="1.016" layer="27" ratio="10"/>
 </element>
 </elements>
@@
 <via x="24.5" y="51.25" extent="1-16" drill="0.35"/>
 <via x="27.25" y="51.25" extent="1-16" drill="0.35"/>
-<contactref element="S1" pad="5"/>
-<contactref element="S1" pad="6"/>
-<contactref element="S1" pad="7"/>
-<contactref element="S1" pad="8"/>
 <contactref element="LED_RING" pad="P$1"/>
-<wire x1="-5.31" y1="-27.5042" x2="-12" y2="-33" width="0" layer="19" extent="1-1"/>
-<wire x1="-2.77" y1="-27.5042" x2="-5.31" y2="-27.5042" width="0" layer="19" extent="1-1"/>
-<wire x1="-0.23" y1="-27.5042" x2="-2.77" y2="-27.5042" width="0" layer="19" extent="1-1"/>
-<wire x1="2.31" y1="-27.5042" x2="-0.23" y2="-27.5042" width="0" layer="19" extent="1-1"/>
-<wire x1="19.46" y1="9.52" x2="2.31" y2="-27.5042" width="0" layer="19" extent="1-1"/>
+<contactref element="FAN" pad="3"/>
+<wire x1="-12" y1="-33" x2="-12.73" y2="-51" width="0" layer="19" extent="1-1"/>
+<wire x1="19.46" y1="9.52" x2="-12" y2="-33" width="0" layer="19" extent="1-1"/>
 </signal>
 <signal name="GND">
@@
 <via x="29.5" y="51.25" extent="1-16" drill="0.35"/>
 <via x="65.25" y="51.25" extent="1-16" drill="0.35"/>
-<contactref element="R1" pad="2"/>
 <contactref element="LED_RING" pad="P$2"/>
-<wire x1="7.0033" y1="-13.1176" x2="-14.5" y2="-33" width="0" layer="19" extent="1-1"/>
-<wire x1="2.77" y1="9.52" x2="7.0033" y2="-13.1176" width="0" layer="19" extent="1-1"/>
+<contactref element="R1" pad="1"/>
+<contactref element="FAN" pad="4"/>
+<wire x1="-14.5" y1="-33" x2="-10.19" y2="-51" width="0" layer="19" extent="1-1"/>
+<wire x1="4.9967" y1="-13.1176" x2="-14.5" y2="-33" width="0" layer="19" extent="1-1"/>
+<wire x1="2.77" y1="9.52" x2="4.9967" y2="-13.1176" width="0" layer="19" extent="1-1"/>
 </signal>
 <signal name="L0M1">
@@
 <wire x1="13.25" y1="35.75" x2="13.41" y2="35.98" width="0.1524" layer="1"/>
 <wire x1="7" y1="12.25" x2="8.01" y2="12.08" width="0.1524" layer="1"/>
-<contactref element="R1" pad="1"/>
-<wire x1="4.9967" y1="-13.1176" x2="4.74" y2="12.13" width="0" layer="19" extent="1-1"/>
+<contactref element="R1" pad="2"/>
+<wire x1="7.0033" y1="-13.1176" x2="8.01" y2="12.08" width="0" layer="19" extent="1-1"/>
 </signal>
 <signal name="12V_PRE">
@@
 <contactref element="RPI5" pad="1"/>
 <contactref element="X1" pad="1"/>
-<wire x1="-17.77" y1="-43" x2="24.5" y2="51.35" width="0" layer="19" extent="1-1"/>
+<contactref element="S1" pad="8"/>
+<contactref element="S1" pad="7"/>
+<contactref element="S1" pad="6"/>
+<contactref element="S1" pad="5"/>
+<wire x1="2.31" y1="-27.5042" x2="24.5" y2="51.35" width="0" layer="19" extent="1-1"/>
+<wire x1="-0.23" y1="-27.5042" x2="2.31" y2="-27.5042" width="0" layer="19" extent="1-1"/>
+<wire x1="-2.77" y1="-27.5042" x2="-0.23" y2="-27.5042" width="0" layer="19" extent="1-1"/>
+<wire x1="-5.31" y1="-27.5042" x2="-2.77" y2="-27.5042" width="0" layer="19" extent="1-1"/>
+<wire x1="-17.77" y1="-43" x2="-5.31" y2="-27.5042" width="0" layer="19" extent="1-1"/>
 </signal>
 <signal name="PWRSIG">
@@
 <wire x1="-15.23" y1="-43" x2="27.04" y2="51.35" width="0" layer="19" extent="1-1"/>
 </signal>
+<signal name="FAN_PWM">
+<contactref element="FAN" pad="1"/>
+<contactref element="RPI5" pad="32"/>
+<wire x1="-17.81" y1="-51" x2="62.6" y2="53.89" width="0" layer="19" extent="1-1"/>
+</signal>
+<signal name="FAN_RPM">
+<contactref element="FAN" pad="2"/>
+<contactref element="RPI5" pad="38"/>
+<wire x1="-15.27" y1="-51" x2="70.22" y2="53.89" width="0" layer="19" extent="1-1"/>
+</signal>
 </signals>
