File: Mk2/Mk2_PCB/hexapod_mk2_v0.0.sch (EAGLE design)
At the start: 16 parts

Commit message: Mk1 cleanup + PCB revisions
Parts:
- removed LEG6: 06-JST-B6B-XH-A, bt_con-jst-xh:06-JST-B6B-XH-A
- added LED_RING: 03-JST-B3B-XH-A, bt_con-jst-xh:03-JST-B3B-XH-A
- added LEG0: 06-JST-B6B-XH-A, bt_con-jst-xh:06-JST-B6B-XH-A
- added R1: MPMT10014001AT1MPM_VIS, MPMT10014001AT1:MPMT10014001AT1MPM_VIS
- added S1: SWS004, smd-special:SWS004
- added X1: JST-XH-02-PIN-LONG-PAD, Rembrandt Electronics - JST XH Connectors v1-0:JST-XH-02-PIN-LONG-PAD
- 100R: value (none) -> 100
- 12V: value (none) -> Blue
- 470R: value (none) -> 470
- 5V: value (none) -> Red
- RPI5: value (none) -> Raspberry Pi
Connections:
- removed net 3V3: RPI5.1
- removed net 3V3_2: RPI5.17
- removed net GPIO10: RPI5.19
- removed net GPIO11: RPI5.23
- removed net GPIO12: RPI5.32
- removed net GPIO13: RPI5.33
- removed net GPIO16: RPI5.36
- removed net GPIO17: RPI5.11
- removed net GPIO18: RPI5.12
- removed net GPIO19: RPI5.35
- removed net GPIO2: RPI5.3
- removed net GPIO20: RPI5.38
- removed net GPIO21: RPI5.40
- removed net GPIO22: RPI5.15
- removed net GPIO23: RPI5.16
- removed net GPIO24: RPI5.18
- removed net GPIO25: RPI5.22
- removed net GPIO26: RPI5.37
- removed net GPIO27: RPI5.13
- removed net GPIO3: RPI5.5
- removed net GPIO4: RPI5.7
- removed net GPIO5: RPI5.29
- removed net GPIO6: RPI5.31
- removed net GPIO7: RPI5.26
- removed net GPIO8: RPI5.24
- removed net GPIO9: RPI5.21
- removed net ID_SC: RPI5.28
- removed net ID_SD: RPI5.27
- removed net L6M1: LEG6-3.1, U$1.19-A5/SCL0
- removed net L6M2: LEG6-4.1, U$1.22-A8/CTX1
- removed net L6M3: LEG6-5.1, U$1.23-A9/CRX1/MCLK1
- removed net L6SIG: LEG6-6.1, U$1.29-TX7
- new net 3.3V: RPI5.1, X1-1.S
- new net D_SW0: RPI5.22, S1.1
- new net D_SW1: RPI5.24, S1.2
- new net D_SW2: RPI5.26, S1.3
- new net D_SW3: RPI5.28, S1.4
- new net L0M1: LEG0-3.1, U$1.2-OUT2
- new net L0M2: LEG0-4.1, U$1.3-LRCLK2
- new net L0M3: LEG0-5.1, U$1.4-BCLK2
- new net L0SIG: LEG0-6.1, U$1.24-A10/TX6/SCL2
- new net LEDSIG: LED_RING-3.1, RPI5.33
- new net PWRSIG: RPI5.3, U$1.0-RX1/CS1/CRX2, X1-2.S
- new net V_DIV: R1.3, U$1.38-A14/CS/IN1
- net 12V: now also R1.1
- net 5V: now also LED_RING-1.1, LEG0-1.1, S1.5, S1.6, S1.7, S1.8; no longer LEG6-1.1
- net GND: now also LED_RING-2.1, LEG0-2.1, R1.2; no longer LEG6-2.1
- net L1M1: now also U$1.5-IN2; no longer U$1.2-OUT2
- net L1M2: now also U$1.6-OUT1D; no longer U$1.3-LRCLK2
- net L1M3: now also U$1.7-RX2/OUT1A; no longer U$1.4-BCLK2
- net L1SIG: now also U$1.25-A11/RX6/SDA2; no longer U$1.24-A10/TX6/SCL2
- net L2M1: now also U$1.8-TX2/IN1; no longer U$1.5-IN2
- net L2M2: now also U$1.9-OUT1C; no longer U$1.6-OUT1D
- net L2M3: now also U$1.10-CS/MQSR; no longer U$1.7-RX2/OUT1A
- net L2SIG: now also U$1.26-A12/MOSI1; no longer U$1.25-A11/RX6/SDA2
- net L3M1: now also U$1.11-MOSI/CTX1; no longer U$1.8-TX2/IN1
- net L3M2: now also U$1.12-MISO/MQSL; no longer U$1.9-OUT1C
- net L3M3: now also U$1.13-SCK/LED; no longer U$1.10-CS/MQSR
- net L3SIG: now also U$1.27-A13/SCK1; no longer U$1.26-A12/MOSI1
- net L4M1: now also U$1.14-A0/TX3/SPDIF_OUT; no longer U$1.11-MOSI/CTX1
- net L4M2: now also U$1.15-A1/RX3/SPDIF_IN; no longer U$1.12-MISO/MQSL
- net L4M3: now also U$1.18-A4/SDA0; no longer U$1.13-SCK/LED
- net L4SIG: now also U$1.28-RX7; no longer U$1.27-A13/SCK1
- net L5M1: now also U$1.19-A5/SCL0; no longer U$1.14-A0/TX3/SPDIF_OUT
- net L5M2: now also U$1.22-A8/CTX1; no longer U$1.15-A1/RX3/SPDIF_IN
- net L5M3: now also U$1.23-A9/CRX1/MCLK1; no longer U$1.18-A4/SDA0
- net L5SIG: now also U$1.29-TX7; no longer U$1.28-RX7
Other:
- moved on the sheet: 100R, 12V, 470R, 5V, BUCK_IN, BUCK_OUT, LEG1-1, LEG1-2, LEG1-3, LEG1-4, LEG1-5, LEG1-6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

Commit message: Update Mk2 Schematic
Parts:
- added FAN: JST-XH-04-PIN-LONG-PAD, Rembrandt Electronics - JST XH Connectors v1-0:JST-XH-04-PIN-LONG-PAD
Connections:
- new net FAN_PWM: FAN-1.S, RPI5.32
- new net FAN_RPM: FAN-2.S, RPI5.38
- net 12V: now also R1.2; no longer R1.1
- net 3.3V: now also S1.5, S1.6, S1.7, S1.8
- net 5V: now also FAN-3.S; no longer S1.5, S1.6, S1.7, S1.8
- net GND: now also FAN-4.S, R1.1; no longer R1.2
