File: Mk2/Mk2_PCB/hexapod_mk2_leg_v0.0.brd (EAGLE design)
At the start: 27 x 22.4 mm, 5 parts

Commit message: update leg pcb
Parts:
- moved LIMIT 16.4 mm to (4.86, 5.60), turned to 180 degrees
- moved S1 16.2 mm to (21.4, 5.40), turned to 180 degrees
- moved S3 8.60 mm to (6.05, 12.6), turned to 180 degrees
- moved MAIN 1.97 mm to (14.1, 20.1), turned to 180 degrees
- moved S2 1.42 mm to (21.5, 12.6), turned to 180 degrees
Connections:
- net 5V: now also MAIN.3, S1.2, S2.2, S3.2; no longer MAIN.1, S1.1, S2.1, S3.1
- net GND: now also MAIN.4, S1.1, S2.1, S3.1; no longer MAIN.2, S1.2, S2.2, S3.2
- net S1SIG: now also MAIN.1; no longer MAIN.3
- net S2SIG: now also MAIN.2; no longer MAIN.4
Routing:
- net GND: track 39.9 -> 0.00 mm
- net 5V: track 29.5 -> 0.00 mm
- net S1SIG: track 8.84 -> 29.1 mm
- net S2SIG: track 11.4 -> 24.6 mm
- net S3SIG: track 17.8 -> 10.3 mm
- net LIMIT: track 14.3 -> 19.9 mm
- added copper zone on layer 1, net 5V
- added copper zone on layer 16, net GND
Other:
- outline, holes or cut-outs redrawn
