File: Mk2/Mk2_PCB/hexapod_mk2_main_v0.0.sch (EAGLE design)
At the start: 21 parts, among them X1 JST-XH-02-PIN-LONG-PAD

Commit message: Finalized main PCB
Parts:
- added U1: 74LVC1T45GW,125TSSOP6_SOT363-2_NEX-M, logic-level-converter:74LVC1T45GW,125TSSOP6_SOT363-2_NEX-M
- 12V: value Blue -> (none)
- 1KΩ: value 470 -> (none)
- 200Ω: value 100 -> (none)
- 5V: value Red -> (none)
- renumbered 100R to 200Ω, 470R to 1KΩ, POWER_SWITCH to E_STOP, X1 to P_BUTTON
Connections:
- new net LEDSIG_CONV: LED_RING-3.1, U1.A
- net 3.3V: now also U1.VCC(B)
- net 5V: now also U1.VCC(A)
- net GND: now also U1.DIR, U1.GND
- net LEDSIG: now also U1.B; no longer LED_RING-3.1

Commit message: board update
Connections:
- net 5V: now also LEG0-3.1, LEG1-3.1, LEG2-3.1, LEG3-3.1, LEG4-3.1, LEG5-3.1; no longer LEG0-1.1, LEG1-1.1, LEG2-1.1, LEG3-1.1, LEG4-1.1, LEG5-1.1
- net GND: now also LEG0-4.1, LEG1-4.1, LEG2-4.1, LEG3-4.1, LEG4-4.1, LEG5-4.1; no longer LEG0-2.1, LEG1-2.1, LEG2-2.1, LEG3-2.1, LEG4-2.1, LEG5-2.1
- net L0M1: now also LEG0-1.1; no longer LEG0-3.1
- net L0M2: now also LEG0-2.1; no longer LEG0-4.1
- net L1M1: now also LEG1-1.1; no longer LEG1-3.1
- net L1M2: now also LEG1-2.1; no longer LEG1-4.1
- net L2M1: now also LEG2-1.1; no longer LEG2-3.1
- net L2M2: now also LEG2-2.1; no longer LEG2-4.1
- net L3M1: now also LEG3-1.1; no longer LEG3-3.1
- net L3M2: now also LEG3-2.1; no longer LEG3-4.1
- net L4M1: now also LEG4-1.1; no longer LEG4-3.1
- net L4M2: now also LEG4-2.1; no longer LEG4-4.1
- net L5M1: now also LEG5-1.1; no longer LEG5-3.1
- net L5M2: now also LEG5-2.1; no longer LEG5-4.1
