File: Mk2/Mk2_PCB/hexapod_mk2_main_v0.0.brd (EAGLE design)
At the start: 80.5 x 61 mm, 21 parts, among them X1 JST-XH-02-PIN-LONG-PAD

Commit message: Finalized main PCB
Parts:
- removed 100R: 100, rcl:R0805
- removed 470R: 470, rcl:R0805
- removed POWER_SWITCH: XT30PW-M, amass:XT30PW-M
- removed X1: JST-XH-02-PIN-LONG-PAD, Rembrandt Electronics - JST XH Connectors v1-0:JST-XH-02-PACKAGE-LONG-PAD
- added 1KΩ, 200Ω: (no value), rcl:R0805
- added E_STOP: XT30PW-M, amass:XT30PW-M
- added P_BUTTON: JST-XH-02-PIN-LONG-PAD, Rembrandt Electronics - JST XH Connectors v1-0:JST-XH-02-PACKAGE-LONG-PAD
- added U1: 74LVC1T45GW,125TSSOP6_SOT363-2_NEX-M, logic-level-converter:TSSOP6_SOT363-2_NEX-M
- 12V: value Blue -> (none)
- 5V: value Red -> (none)
- moved FAN 98.7 mm to (68.0, 4.00)
- moved S1 78.3 mm to (47.0, 29.5)
- moved LED_RING 57.9 mm to (30.0, 4.00)
- moved R1 43.4 mm to (24.0, 27.5)
- moved 12V 18.4 mm to (21.5, 7.50), turned to 180 degrees
- moved LEG5 9.66 mm to (26.9, 12.4)
- moved LEG4 9.12 mm to (46.6, 12.4)
- moved LEG3 9.00 mm to (66.4, 12.4)
- moved U$1 5.50 mm to (47.3, 29.4)
- moved LEG0 3.20 mm to (26.9, 42.5)
- moved LEG1 2.50 mm to (46.6, 42.5)
- moved 5V 2.46 mm to (17.0, 7.50), turned to 180 degrees
- moved BUCK_OUT 2.09 mm to (11.4, 53.1)
- moved BUCK_IN 2.06 mm to (11.4, 39.0)
- moved LEG2 2.00 mm to (66.3, 42.5)
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Connections:
- new net LEDSIG_CONV: LED_RING.P$3, U1.3
- net 12V: now also E_STOP.-; no longer POWER_SWITCH.-
- net 12V_PRE: now also E_STOP.+; no longer POWER_SWITCH.+
- net 3.3V: now also P_BUTTON.1, U1.6; no longer X1.1
- net 5V: now also U1.1
- net GND: now also 1KΩ.1, 200Ω.1, U1.2, U1.5; no longer 100R.1, 470R.1
- net LEDSIG: now also U1.4; no longer LED_RING.P$3
- net N$1: now also 200Ω.2; no longer 100R.2
- net N$2: now also 1KΩ.2; no longer 470R.2
- net PWRSIG: now also P_BUTTON.2; no longer X1.2
Routing:
- net PWRSIG: track 0.00 -> 138.2 mm
- net 3.3V: track 0.00 -> 93.1 mm, vias 0 -> 2
- net FAN_PWM: track 0.00 -> 76.7 mm
- net LEDSIG: track 0.00 -> 59.8 mm, vias 0 -> 2
- net 5V: track 187.7 -> 247.3 mm, vias 4 -> 1
- net FAN_RPM: track 0.00 -> 59.5 mm
- net D_SW2: track 0.00 -> 54.4 mm
- net D_SW3: track 0.00 -> 46.9 mm
- net GND: track 345.4 -> 300.2 mm, vias 11 -> 0
- net D_SW0: track 0.00 -> 40.8 mm
- net D_SW1: track 0.00 -> 35.6 mm, vias 0 -> 1
- net L0M3: track 43.2 -> 76.7 mm, vias 1 -> 0
- net LEDSIG_CONV: track 0.00 -> 29.3 mm, vias 0 -> 1
- net L1M3: track 41.3 -> 17.0 mm
- net L1M1: track 39.1 -> 17.1 mm
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- added copper zone on layer 15, net 5V
- added copper zone on layer 2, net GND
Other:
- board size 80.5 x 61 mm -> 84.5 x 61 mm
- board text added: "VOLT_DIV"

Commit message: board update
Connections:
- net 5V: now also LEG0.P$3, LEG1.P$3, LEG2.P$3, LEG3.P$3, LEG4.P$3, LEG5.P$3; no longer LEG0.P$1, LEG1.P$1, LEG2.P$1, LEG3.P$1, LEG4.P$1, LEG5.P$1
- net GND: now also LEG0.P$4, LEG1.P$4, LEG2.P$4, LEG3.P$4, LEG4.P$4, LEG5.P$4; no longer LEG0.P$2, LEG1.P$2, LEG2.P$2, LEG3.P$2, LEG4.P$2, LEG5.P$2
- net L0M1: now also LEG0.P$1; no longer LEG0.P$3
- net L0M2: now also LEG0.P$2; no longer LEG0.P$4
- net L1M1: now also LEG1.P$1; no longer LEG1.P$3
- net L1M2: now also LEG1.P$2; no longer LEG1.P$4
- net L2M1: now also LEG2.P$1; no longer LEG2.P$3
- net L2M2: now also LEG2.P$2; no longer LEG2.P$4
- net L3M1: now also LEG3.P$1; no longer LEG3.P$3
- net L3M2: now also LEG3.P$2; no longer LEG3.P$4
- net L4M1: now also LEG4.P$1; no longer LEG4.P$3
- net L4M2: now also LEG4.P$2; no longer LEG4.P$4
- net L5M1: now also LEG5.P$1; no longer LEG5.P$3
- net L5M2: now also LEG5.P$2; no longer LEG5.P$4
Routing:
- net 5V: track 247.3 -> 225.3 mm
- net GND: track 300.2 -> 299.2 mm
Other:
- board text added: "Main Board V2.0 June 2024"

Commit message: auto route main board. add silkscreens to both
Parts:
- moved R1 0.29 mm to (24.0, 27.8)
Routing:
- net L3M1: track 33.8 -> 65.9 mm
- net L0M3: track 76.7 -> 51.8 mm
- net L5M2: track 68.0 -> 43.8 mm
- net FAN_PWM: track 76.7 -> 54.4 mm
- net D_SW2: track 54.4 -> 33.3 mm, vias 0 -> 1
- net GND: track 299.2 -> 319.9 mm
- net L0M1: track 64.5 -> 45.4 mm
- net 3.3V: track 93.1 -> 110.2 mm, vias 2 -> 3
- net PWRSIG: track 138.2 -> 123.9 mm
- net LEDSIG: track 59.8 -> 73.9 mm, vias 2 -> 0
- net L5M1: track 49.3 -> 36.2 mm
- net 12V: track 50.4 -> 61.5 mm, vias 2 -> 1
- net D_SW3: track 46.9 -> 37.8 mm
- net L3M2: track 34.1 -> 42.9 mm, vias 0 -> 1
- net RPI_TX: track 51.8 -> 60.5 mm
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Other:
- board text added: "+"
- board text added: "Main Board Mk 2, V1.0 June 2024"
- board text added: "VCC_CONV"
- board text added: "⏚"
- board text removed: "Main Board V2.0 June 2024"
