File: mk2/electronics/mainboard/v1.0/hexapod_mk2_main_v1.0.brd (EAGLE design)
At the start: 84.5 x 61 mm, 22 parts, among them U1 74LVC1T45GW,125TSSOP6_SOT363-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

Commit message: Update mainboard schematic v1.0
Parts:
- removed BUCK_IN, BUCK_OUT: XT30PW-M, amass:XT30PW-M
- removed S1: SWS004, smd-special:SMS-004
- added DFR0753: DFR0753, DFR0753:DFR0753
- added FUSE_HOLDER: 3555-2, 3555-2:FUSE_3555-2
- added U2: SN74LVC1T45DBVR, SN74LVC1T45DBVR:SOT95P280X145-6N
- E_STOP: value XT30PW-M -> XT60PW-M; device amass:XT30PW-M -> amass:XT60PW-M
- moved E_STOP 38.1 mm to (-13.2, -21.6), turned to 0 degrees
- renumbered 12V to 2S
Connections:
- removed net 12V: 2S.A, BUCK_IN.+, E_STOP.-, R1.2
- removed net 12V_PRE: BATTERY.+, E_STOP.+
- removed net D_SW0: RPI5.22, S1.1
- removed net D_SW1: RPI5.24, S1.2
- removed net D_SW2: RPI5.26, S1.3
- removed net D_SW3: RPI5.28, S1.4
- new net 2S_BAT: BATTERY.+, E_STOP.-
- new net 2S_ESTOP: E_STOP.+, FUSE_HOLDER.1_1, FUSE_HOLDER.1_2
- new net 2S_PROT: 2S.A, DFR0753.VIN, FUSE_HOLDER.2_1, FUSE_HOLDER.2_2, LEG0.P$3, LEG1.P$3, LEG2.P$3, LEG3.P$3, LEG4.P$3, LEG5.P$3, R1.2
- net 3.3V: now also U2.6; no longer P_BUTTON.1, S1.5, S1.6, S1.7, S1.8
- net 5V: now also DFR0753.VOUT, U2.1; no longer BUCK_OUT.+, LEG0.P$3, LEG1.P$3, LEG2.P$3, LEG3.P$3, LEG4.P$3, LEG5.P$3
- net GND: now also DFR0753.GND, P_BUTTON.1, U2.2, U2.5; no longer BUCK_IN.-, BUCK_OUT.-
- net LEDSIG: now also U2.4
- net LEDSIG_CONV: now also U2.3
- net PWRSIG: now also RPI5.11; no longer RPI5.3, U$1.0-RX1/CS1/CRX2
Routing:
- net PWRSIG: track 123.9 -> 60.6 mm
- net 12V: track 61.5 -> 0.00 mm, vias 1 -> 0
- net 3.3V: track 110.2 -> 65.0 mm, vias 3 -> 2
- net D_SW3: track 37.8 -> 0.00 mm
- net 2S_PROT: track 0.00 -> 36.1 mm, vias 0 -> 1
- net D_SW0: track 33.4 -> 0.00 mm, vias 1 -> 0
- net D_SW2: track 33.3 -> 0.00 mm, vias 1 -> 0
- net D_SW1: track 31.7 -> 0.00 mm, vias 1 -> 0
- net 12V_PRE: track 25.0 -> 0.00 mm

Commit message: fix board sever
Parts:
- removed DFR0753: DFR0753, DFR0753:DFR0753
- removed FUSE_HOLDER: 3555-2, 3555-2:FUSE_3555-2
- removed U2: SN74LVC1T45DBVR, SN74LVC1T45DBVR:SOT95P280X145-6N
- added BUCK_IN, BUCK_OUT: XT30PW-M, amass:XT30PW-M
- added S1: SWS004, smd-special:SMS-004
- E_STOP: value XT60PW-M -> XT30PW-M; device amass:XT60PW-M -> amass:XT30PW-M
- moved E_STOP 38.1 mm to (11.4, 7.49), turned to 90 degrees
- renumbered 2S to 12V
Connections:
- removed net 2S_BAT: BATTERY.+, E_STOP.-
- removed net 2S_ESTOP: E_STOP.+, FUSE_HOLDER.1_1, FUSE_HOLDER.1_2
- removed net 2S_PROT: 12V.A, DFR0753.VIN, FUSE_HOLDER.2_1, FUSE_HOLDER.2_2, LEG0.P$3, LEG1.P$3, LEG2.P$3, LEG3.P$3, LEG4.P$3, LEG5.P$3, R1.2
- new net 12V: 12V.A, BUCK_IN.+, E_STOP.-, R1.2
- new net 12V_PRE: BATTERY.+, E_STOP.+
- new net D_SW0: RPI5.22, S1.1
- new net D_SW1: RPI5.24, S1.2
- new net D_SW2: RPI5.26, S1.3
- new net D_SW3: RPI5.28, S1.4
- net 3.3V: now also P_BUTTON.1, S1.5, S1.6, S1.7, S1.8; no longer U2.6
- net 5V: now also BUCK_OUT.+, LEG0.P$3, LEG1.P$3, LEG2.P$3, LEG3.P$3, LEG4.P$3, LEG5.P$3; no longer DFR0753.VOUT, U2.1
- net GND: now also BUCK_IN.-, BUCK_OUT.-; no longer DFR0753.GND, P_BUTTON.1, U2.2, U2.5
- net LEDSIG: no longer U2.4
- net LEDSIG_CONV: no longer U2.3
- net PWRSIG: now also RPI5.3, U$1.0-RX1/CS1/CRX2; no longer RPI5.11
Routing:
- net PWRSIG: track 60.6 -> 123.9 mm
- net 12V: track 0.00 -> 61.5 mm, vias 0 -> 1
- net 3.3V: track 65.0 -> 110.2 mm, vias 2 -> 3
- net D_SW3: track 0.00 -> 37.8 mm
- net 2S_PROT: track 36.1 -> 0.00 mm, vias 1 -> 0
- net D_SW0: track 0.00 -> 33.4 mm, vias 0 -> 1
- net D_SW2: track 0.00 -> 33.3 mm, vias 0 -> 1
- net D_SW1: track 0.00 -> 31.7 mm, vias 0 -> 1
- net 12V_PRE: track 0.00 -> 25.0 mm
