File: mk2/electronics/mainboard/v1.0/hexapod_mk2_main_v1.0.sch (EAGLE design)
At the start: 21 parts

Commit message: fix board sever
Parts:
- removed DFR0753: DFR0753, DFR0753:DFR0753
- removed FUSE_HOLDER: 3555-2, 3555-2:3555-2
- removed LED_SIGNAL_VOLTAGE: SN74LVC1T45DBVR, SN74LVC1T45DBVR:SN74LVC1T45DBVR
- added BUCK_IN, BUCK_OUT: XT30PW-M, amass:XT30PW-M
- added S1: SWS004, smd-special:SWS004
- added U1: 74LVC1T45GW,125TSSOP6_SOT363-2_NEX-M, logic-level-converter:74LVC1T45GW,125TSSOP6_SOT363-2_NEX-M
- E_STOP: value XT60PW-M -> XT30PW-M; device amass:XT60PW-M -> amass:XT30PW-M
- renumbered 2S to 12V, 680Ω to 1KΩ
Connections:
- removed net 2S_BAT: BATTERY.+, E_STOP.-
- removed net 2S_ESTOP: E_STOP.+, FUSE_HOLDER.1
- removed net 2S_PROT: 12V.A, DFR0753.VIN, FUSE_HOLDER.2, LEG0-3.1, LEG1-3.1, LEG2-3.1, LEG3-3.1, LEG4-3.1, LEG5-3.1, R1.2
- new net 12V: 12V.A, BUCK_IN.+, E_STOP.-, R1.2
- new net 12V_PRE: BATTERY.+, E_STOP.+
- new net D_SW0: RPI5.22, S1.1
- new net D_SW1: RPI5.24, S1.2
- new net D_SW2: RPI5.26, S1.3
- new net D_SW3: RPI5.28, S1.4
- net 3.3V: now also P_BUTTON-1.S, S1.5, S1.6, S1.7, S1.8, U1.VCC(B); no longer LED_SIGNAL_VOLTAGE.VCCB
- net 5V: now also BUCK_OUT.+, LEG0-3.1, LEG1-3.1, LEG2-3.1, LEG3-3.1, LEG4-3.1, LEG5-3.1, U1.VCC(A); no longer DFR0753.VOUT, LED_SIGNAL_VOLTAGE.VCCA
- net GND: now also BUCK_IN.-, BUCK_OUT.-, U1.DIR, U1.GND; no longer DFR0753.GND, LED_SIGNAL_VOLTAGE.DIR, LED_SIGNAL_VOLTAGE.GND, P_BUTTON-1.S
- net LEDSIG: now also RPI5.33, U1.B; no longer LED_SIGNAL_VOLTAGE.B, RPI5.19
- net LEDSIG_CONV: now also U1.A; no longer LED_SIGNAL_VOLTAGE.A
- net PWRSIG: now also RPI5.3, U$1.0-RX1/CS1/CRX2; no longer RPI5.11
Other:
- moved on the sheet: FAN-1, FAN-2, FAN-3, FAN-4, P_BUTTON-1, P_BUTTON-2
