File: mk2/electronics/mainboard/v2.0/hexapod_mk2_main_v2.0.sch (EAGLE design)
At the start: 22 parts, among them U1 74LVC1T45GW,125TSSOP6_SOT363-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

Commit message: fix board sever
Parts:
- removed BUCK_IN, BUCK_OUT: XT30PW-M, amass:XT30PW-M
- removed S1: SWS004, smd-special:SWS004
- removed U1: 74LVC1T45GW,125TSSOP6_SOT363-2_NEX-M, logic-level-converter:74LVC1T45GW,125TSSOP6_SOT363-2_NEX-M
- added DFR0753: DFR0753, DFR0753:DFR0753
- added FUSE_HOLDER: 3555-2, 3555-2:3555-2
- added U2: SN74LVC1T45DBVR, SN74LVC1T45DBVR:SN74LVC1T45DBVR
- E_STOP: value XT30PW-M -> XT60PW-M; device amass:XT30PW-M -> amass:XT60PW-M
- renumbered 12V to 2S, 1KΩ to 680Ω
Connections:
- removed net 12V: 2S.A, BUCK_IN.+, E_STOP.-, R1.2
- removed net 12V_PRE: BATTERY.+, E_STOP.+
- removed net D_SW0: RPI5.22, S1.1
- removed net D_SW1: RPI5.24, S1.2
- removed net D_SW2: RPI5.26, S1.3
- removed net D_SW3: RPI5.28, S1.4
- new net 2S_BAT: BATTERY.+, E_STOP.-
- new net 2S_ESTOP: E_STOP.+, FUSE_HOLDER.1
- new net 2S_PROT: 2S.A, DFR0753.VIN, FUSE_HOLDER.2, LEG0-3.1, LEG1-3.1, LEG2-3.1, LEG3-3.1, LEG4-3.1, LEG5-3.1, R1.2
- net 3.3V: now also U2.VCCB; no longer P_BUTTON-1.S, S1.5, S1.6, S1.7, S1.8, U1.VCC(B)
- net 5V: now also DFR0753.VOUT, U2.VCCA; no longer BUCK_OUT.+, LEG0-3.1, LEG1-3.1, LEG2-3.1, LEG3-3.1, LEG4-3.1, LEG5-3.1, U1.VCC(A)
- net GND: now also DFR0753.GND, P_BUTTON-1.S, U2.DIR, U2.GND; no longer BUCK_IN.-, BUCK_OUT.-, U1.DIR, U1.GND
- net LEDSIG: now also RPI5.19, U2.B; no longer RPI5.33, U1.B
- net LEDSIG_CONV: now also U2.A; no longer U1.A
- net PWRSIG: now also RPI5.11; no longer RPI5.3, U$1.0-RX1/CS1/CRX2
Other:
- moved on the sheet: FAN-1, FAN-2, FAN-3, FAN-4, P_BUTTON-1, P_BUTTON-2
