File: mk2/electronics/mainboard/v2.0/hexapod_mk2_main_v2.0.sch (EAGLE design)
At the start: 21 parts, among them U2 SN74LVC1T45DBVR

Commit message: ordered
Parts:
- removed FUSE_HOLDER: 3555-2, 3555-2:3555-2
- added F1: 3557-2, 3557-2:3557-2
Connections:
- net 2S_BAT: now also E_STOP.+; no longer E_STOP.-
- net 2S_ESTOP: now also E_STOP.-, F1.1; no longer E_STOP.+, FUSE_HOLDER.1
- net 2S_PROT: now also F1.2; no longer FUSE_HOLDER.2
Changed lines of the file:
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@@
 <part name="2S" library="led" library_urn="urn:adsk.eagle:library:259" deviceset="LED" device="CHIPLED_0805" package3d_urn="urn:adsk.eagle:package:15821/2"/>
 <part name="E_STOP" library="amass" deviceset="XT60" device="PW-M"/>
-<part name="FUSE_HOLDER" library="3555-2" deviceset="3555-2" device=""/>
 <part name="DFR0753" library="DFR0753" deviceset="DFR0753" device=""/>
 <part name="U2" library="SN74LVC1T45DBVR" deviceset="SN74LVC1T45DBVR" device=""/>
+<part name="F1" library="3557-2" deviceset="3557-2" device=""/>
 </parts>
 <sheets>
@@
 <attribute name="NAME" x="-156.21" y="93.472" size="1.778" layer="95"/>
 </instance>
-<instance part="FUSE_HOLDER" gate="G$1" x="-109.22" y="86.36" smashed="yes">
-<attribute name="NAME" x="-116.84" y="90.17" size="1.778" layer="95"/>
-<attribute name="VALUE" x="-116.84" y="82.55" size="1.778" layer="96" align="top-left"/>
-</instance>
 <instance part="DFR0753" gate="G$1" x="-60.96" y="91.44" smashed="yes"/>
 <instance part="U2" gate="A" x="-20.32" y="-35.56" smashed="yes">
 <attribute name="NAME" x="-33.02" y="-21.86" size="2.0828" layer="95" ratio="10" rot="SR0"/>
 <attribute name="VALUE" x="-33.02" y="-52.26" size="2.0828" layer="96" ratio="10" rot="SR0"/>
+</instance>
+<instance part="F1" gate="G$1" x="-109.22" y="86.36" smashed="yes">
+<attribute name="NAME" x="-111.76" y="91.44" size="1.27" layer="95"/>
+<attribute name="VALUE" x="-111.76" y="81.28" size="1.27" layer="96"/>
 </instance>
 </instances>
@@
 </segment>
 <segment>
+<pinref part="E_STOP" gate="G$1" pin="+"/>
+<wire x1="-147.32" y1="88.9" x2="-144.78" y2="88.9" width="0.1524" layer="91"/>
+<label x="-144.78" y="88.9" size="1.778" layer="95"/>
+</segment>
+</net>
+<net name="2S_PROT" class="0">
+<segment>
+<wire x1="-101.6" y1="86.36" x2="-93.98" y2="86.36" width="0.1524" layer="91"/>
+<label x="-93.98" y="86.36" size="1.778" layer="95"/>
+<pinref part="F1" gate="G$1" pin="2"/>
+</segment>
+<segment>
+<wire x1="-144.78" y1="66.04" x2="-144.78" y2="68.58" width="0.1524" layer="91"/>
+<label x="-144.78" y="68.58" size="1.778" layer="95"/>
+<pinref part="2S" gate="G$1" pin="A"/>
+</segment>
+<segment>
+<pinref part="LEG0" gate="-3" pin="1"/>
+<wire x1="-182.88" y1="63.5" x2="-185.42" y2="63.5" width="0.1524" layer="91"/>
+<label x="-190.5" y="63.5" size="1.778" layer="95"/>
+</segment>
+<segment>
+<pinref part="LEG1" gate="-3" pin="1"/>
+<wire x1="-182.88" y1="43.18" x2="-185.42" y2="43.18" width="0.1524" layer="91"/>
+<label x="-190.5" y="43.18" size="1.778" layer="95"/>
+</segment>
+<segment>
+<pinref part="LEG2" gate="-3" pin="1"/>
+<wire x1="-182.88" y1="22.86" x2="-185.42" y2="22.86" width="0.1524" layer="91"/>
+<label x="-190.5" y="22.86" size="1.778" layer="95"/>
+</segment>
+<segment>
+<pinref part="LEG3" gate="-3" pin="1"/>
+<wire x1="-182.88" y1="2.54" x2="-185.42" y2="2.54" width="0.1524" layer="91"/>
+<label x="-190.5" y="2.54" size="1.778" layer="95"/>
+</segment>
+<segment>
+<pinref part="LEG4" gate="-3" pin="1"/>
+<wire x1="-182.88" y1="-17.78" x2="-185.42" y2="-17.78" width="0.1524" layer="91"/>
+<label x="-190.5" y="-17.78" size="1.778" layer="95"/>
+</segment>
+<segment>
+<pinref part="LEG5" gate="-3" pin="1"/>
+<wire x1="-182.88" y1="-38.1" x2="-185.42" y2="-38.1" width="0.1524" layer="91"/>
+<label x="-190.5" y="-38.1" size="1.778" layer="95"/>
+</segment>
+<segment>
+<pinref part="DFR0753" gate="G$1" pin="VIN"/>
+<wire x1="-71.12" y1="83.82" x2="-76.2" y2="83.82" width="0.1524" layer="91"/>
+<label x="-83.82" y="83.82" size="1.778" layer="95"/>
+</segment>
+<segment>
+<pinref part="R1" gate="A" pin="2"/>
+<wire x1="-149.86" y1="2.54" x2="-152.4" y2="2.54" width="0.1524" layer="91"/>
+<label x="-154.94" y="2.54" size="1.778" layer="95"/>
+</segment>
+</net>
+<net name="2S_ESTOP" class="0">
+<segment>
+<wire x1="-116.84" y1="86.36" x2="-127" y2="86.36" width="0.1524" layer="91"/>
+<label x="-127" y="83.82" size="1.778" layer="95"/>
+<pinref part="F1" gate="G$1" pin="1"/>
+</segment>
+<segment>
 <pinref part="E_STOP" gate="G$1" pin="-"/>
 <wire x1="-147.32" y1="83.82" x2="-144.78" y2="83.82" width="0.1524" layer="91"/>
@@
 </segment>
 </net>
-<net name="2S_PROT" class="0">
-<segment>
-<pinref part="FUSE_HOLDER" gate="G$1" pin="2"/>
-<wire x1="-99.06" y1="86.36" x2="-93.98" y2="86.36" width="0.1524" layer="91"/>
-<label x="-93.98" y="86.36" size="1.778" layer="95"/>
-</segment>
-<segment>
-<wire x1="-144.78" y1="66.04" x2="-144.78" y2="68.58" width="0.1524" layer="91"/>
-<label x="-144.78" y="68.58" size="1.778" layer="95"/>
-<pinref part="2S" gate="G$1" pin="A"/>
-</segment>
-<segment>
-<pinref part="LEG0" gate="-3" pin="1"/>
-<wire x1="-182.88" y1="63.5" x2="-185.42" y2="63.5" width="0.1524" layer="91"/>
-<label x="-190.5" y="63.5" size="1.778" layer="95"/>
-</segment>
-<segment>
-<pinref part="LEG1" gate="-3" pin="1"/>
-<wire x1="-182.88" y1="43.18" x2="-185.42" y2="43.18" width="0.1524" layer="91"/>
-<label x="-190.5" y="43.18" size="1.778" layer="95"/>
-</segment>
-<segment>
-<pinref part="LEG2" gate="-3" pin="1"/>
-<wire x1="-182.88" y1="22.86" x2="-185.42" y2="22.86" width="0.1524" layer="91"/>
-<label x="-190.5" y="22.86" size="1.778" layer="95"/>
-</segment>
-<segment>
-<pinref part="LEG3" gate="-3" pin="1"/>
-<wire x1="-182.88" y1="2.54" x2="-185.42" y2="2.54" width="0.1524" layer="91"/>
-<label x="-190.5" y="2.54" size="1.778" layer="95"/>
-</segment>
-<segment>
-<pinref part="LEG4" gate="-3" pin="1"/>
-<wire x1="-182.88" y1="-17.78" x2="-185.42" y2="-17.78" width="0.1524" layer="91"/>
-<label x="-190.5" y="-17.78" size="1.778" layer="95"/>
-</segment>
-<segment>
-<pinref part="LEG5" gate="-3" pin="1"/>
-<wire x1="-182.88" y1="-38.1" x2="-185.42" y2="-38.1" width="0.1524" layer="91"/>
-<label x="-190.5" y="-38.1" size="1.778" layer="95"/>
-</segment>
-<segment>
-<pinref part="DFR0753" gate="G$1" pin="VIN"/>
-<wire x1="-71.12" y1="83.82" x2="-76.2" y2="83.82" width="0.1524" layer="91"/>
-<label x="-83.82" y="83.82" size="1.778" layer="95"/>
-</segment>
-<segment>
-<pinref part="R1" gate="A" pin="2"/>
-<wire x1="-149.86" y1="2.54" x2="-152.4" y2="2.54" width="0.1524" layer="91"/>
-<label x="-154.94" y="2.54" size="1.778" layer="95"/>
-</segment>
-</net>
-<net name="2S_ESTOP" class="0">
-<segment>
-<pinref part="E_STOP" gate="G$1" pin="+"/>
-<wire x1="-147.32" y1="88.9" x2="-144.78" y2="88.9" width="0.1524" layer="91"/>
-<label x="-144.78" y="88.9" size="1.778" layer="95"/>
-</segment>
-<segment>
-<pinref part="FUSE_HOLDER" gate="G$1" pin="1"/>
-<wire x1="-119.38" y1="86.36" x2="-127" y2="86.36" width="0.1524" layer="91"/>
-<label x="-127" y="83.82" size="1.778" layer="95"/>
-</segment>
-</net>
