File: mk2/electronics/mainboard/v2.0/hexapod_mk2_main_v2.0.brd (EAGLE design)
At the start: 89 x 61 mm, 21 parts, among them U2 SN74LVC1T45DBVR

Commit message: ordered
Parts:
- removed FUSE_HOLDER: 3555-2, 3555-2:FUSE_3555-2
- added F1: 3557-2, 3557-2:FUSE_3557-2
- moved E_STOP 0.75 mm to (16.3, 12.1)
- moved BATTERY 0.71 mm to (16.2, 29.9)
Connections:
- net 2S_BAT: now also E_STOP.+; no longer E_STOP.-
- net 2S_ESTOP: now also E_STOP.-, F1.1_1, F1.1_2; no longer E_STOP.+, FUSE_HOLDER.1_1, FUSE_HOLDER.1_2
- net 2S_PROT: now also F1.2_1, F1.2_2; no longer FUSE_HOLDER.2_1, FUSE_HOLDER.2_2
Routing:
- net 2S_BAT: track 28.0 -> 71.0 mm
- net 2S_ESTOP: track 17.5 -> 31.3 mm
- net GND: track 52.9 -> 48.0 mm
- net 2S_PROT: track 33.8 -> 35.1 mm
Other:
- board text added: "Main Board Mk 2, V2.1 January 2025"
- board text removed: "Main Board Mk 2, V2.0 November 2024"
Changed lines of the file:
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@@
 <drawing>
 <settings>
-<setting alwaysvectorfont="no"/>
+<setting alwaysvectorfont="yes"/>
 <setting verticaltext="up"/>
 </settings>
@@
 <hole x="87.991" y="4.078" drill="3"/>
 <text x="31.361" y="24.928" size="1.016" layer="21">VOLT_DIV</text>
-<text x="63.492" y="57.954" size="1.5" layer="21" rot="SR0" align="center-left">Main Board Mk 2, V2.0
-November 2024</text>
+<text x="63.492" y="57.954" size="1.5" layer="21" rot="SR0" align="center-left">Main Board Mk 2, V2.1
+January 2025</text>
 <rectangle x1="59.6375" y1="22.4055" x2="59.6895" y2="22.4185" layer="22" rot="R180"/>
 <rectangle x1="59.6115" y1="22.4185" x2="59.6895" y2="22.4315" layer="22" rot="R180"/>
@@
 <attribute name="VALUE" x="26.537" y="9.108" size="1.27" layer="27" rot="R270"/>
 </element>
-<element name="BATTERY" library="amass" package="XT60PW-M" value="XT60PW-M" x="15.5" y="29.857" smashed="yes" rot="R90">
-<attribute name="NAME" x="20.2" y="25.057" size="1.778" layer="25" rot="R90"/>
-<attribute name="VALUE" x="-0.8" y="24.857" size="1.778" layer="27" rot="R90"/>
+<element name="BATTERY" library="amass" package="XT60PW-M" value="XT60PW-M" x="16.215" y="29.857" smashed="yes" rot="R90">
+<attribute name="NAME" x="20.915" y="25.057" size="1.778" layer="25" rot="R90"/>
+<attribute name="VALUE" x="-0.085" y="24.857" size="1.778" layer="27" rot="R90"/>
 </element>
 <element name="LEG0" library="bt_con-jst-xh" package="B6B-XH" value="06-JST-B6B-XH-A" x="37.401" y="42.588" smashed="yes">
@@
 <attribute name="VALUE" x="29.386" y="9.108" size="1.27" layer="27" rot="R270"/>
 </element>
-<element name="E_STOP" library="amass" package="XT60PW-M" value="XT60PW-M" x="15.5" y="12.116" smashed="yes" rot="R90">
-<attribute name="NAME" x="20.2" y="7.316" size="1.778" layer="25" rot="R90"/>
-<attribute name="VALUE" x="-0.8" y="7.116" size="1.778" layer="27" rot="R90"/>
-</element>
-<element name="FUSE_HOLDER" library="3555-2" package="FUSE_3555-2" value="3555-2" x="23.777" y="19.929" smashed="yes" rot="R90">
-<attribute name="MANUFACTURER" value="Keystone" x="23.777" y="19.929" size="1.778" layer="27" rot="R90" display="off"/>
-<attribute name="MAXIMUM_PACKAGE_HEIGHT" value="11.6mm" x="23.777" y="19.929" size="1.778" layer="27" rot="R90" display="off"/>
-<attribute name="NAME" x="27.484" y="13.553" size="1.27" layer="25" rot="R90"/>
-<attribute name="PARTREV" value="A" x="23.777" y="19.929" size="1.778" layer="27" rot="R90" display="off"/>
-<attribute name="SNAPEDA_PN" value="3555-2" x="23.777" y="19.929" size="1.778" layer="27" rot="R90" display="off"/>
-<attribute name="STANDARD" value="Manufacturer Recommendations" x="23.777" y="19.929" size="1.778" layer="27" rot="R90" display="off"/>
-<attribute name="VALUE" x="27.977" y="1.944" size="1.27" layer="27" rot="R90" align="top-left"/>
+<element name="E_STOP" library="amass" package="XT60PW-M" value="XT60PW-M" x="16.254" y="12.116" smashed="yes" rot="R90">
+<attribute name="NAME" x="20.954" y="7.316" size="1.778" layer="25" rot="R90"/>
+<attribute name="VALUE" x="-0.046" y="7.116" size="1.778" layer="27" rot="R90"/>
 </element>
 <element name="DFR0753" library="DFR0753" package="DFR0753" value="DFR0753" x="16.159" y="49.517" smashed="yes" rot="R90">
@@
 </element>
 <element name="U2" library="SN74LVC1T45DBVR" package="SOT95P280X145-6N" value="SN74LVC1T45DBVR" x="34.554" y="31.824" smashed="yes"/>
+<element name="F1" library="3557-2" package="FUSE_3557-2" value="3557-2" x="24.258" y="19.76" smashed="yes" rot="R90">
+<attribute name="MANUFACTURER" value="Keystone" x="24.258" y="19.76" size="1.778" layer="27" rot="R90" display="off"/>
+<attribute name="MAXIMUM_PACKAGE_HEIGHT" value="7.37mm" x="24.258" y="19.76" size="1.778" layer="27" rot="R90" display="off"/>
+<attribute name="NAME" x="20.448" y="9.6" size="1.27" layer="25" rot="R90"/>
+<attribute name="PARTREV" value="D" x="24.258" y="19.76" size="1.778" layer="27" rot="R90" display="off"/>
+<attribute name="SNAPEDA_PN" value="3557-2" x="24.258" y="19.76" size="1.778" layer="27" rot="R90" display="off"/>
+<attribute name="STANDARD" value="Manufacturer Recommendation" x="24.258" y="19.76" size="1.778" layer="27" rot="R90" display="off"/>
+<attribute name="VALUE" x="29.338" y="9.6" size="1.27" layer="27" rot="R90"/>
+</element>
 </elements>
 <signals>
@@
 <vertex x="-4.641" y="65.052"/>
 </polygon>
-<wire x1="19.909" y1="41.017" x2="18.137" y2="41.017" width="2" layer="1"/>
-<wire x1="18.137" y1="41.017" x2="11.167" y2="34.047" width="2" layer="1"/>
-<wire x1="11.167" y1="34.047" x2="11.167" y2="30.59" width="2" layer="1"/>
-<wire x1="11.167" y1="30.59" x2="15.5" y2="26.257" width="2" layer="1"/>
 <wire x1="33.5956" y1="29.8429" x2="33.5956" y2="26.805" width="0.1524" layer="1"/>
 <wire x1="34.3104" y1="30.5577" x2="33.5956" y2="29.8429" width="0.1524" layer="1"/>
@@
 <wire x1="35.9187" y1="31.9873" x2="35.809" y2="31.824" width="0.1524" layer="1"/>
 <wire x1="36.2761" y1="42.5306" x2="36.151" y2="42.588" width="0.1524" layer="1"/>
+<wire x1="16.215" y1="26.257" x2="19.909" y2="29.951" width="2.5" layer="1"/>
+<wire x1="19.909" y1="29.951" x2="19.909" y2="41.017" width="2.5" layer="1"/>
 </signal>
 <signal name="L0M1">
@@
 <signal name="2S_BAT">
 <contactref element="BATTERY" pad="+"/>
-<contactref element="E_STOP" pad="-"/>
-<wire x1="15.5" y1="33.457" x2="18.992" y2="29.965" width="3" layer="1"/>
-<wire x1="18.992" y1="29.965" x2="19.058" y2="29.965" width="3" layer="1"/>
-<wire x1="19.058" y1="29.965" x2="19.058" y2="27.80855625" width="3" layer="1"/>
-<wire x1="19.058" y1="27.80855625" x2="19.113" y2="27.75355625" width="3" layer="1"/>
-<wire x1="19.113" y1="27.75355625" x2="19.113" y2="12.129" width="3" layer="1"/>
-<wire x1="19.113" y1="12.129" x2="15.5" y2="8.516" width="3" layer="1"/>
+<contactref element="E_STOP" pad="+"/>
+<wire x1="16.215" y1="33.457" x2="15.452" y2="33.457" width="4" layer="1"/>
+<wire x1="15.452" y1="33.457" x2="15.431" y2="33.436" width="4" layer="1"/>
+<wire x1="15.452" y1="33.457" x2="13.769" y2="33.457" width="5.5" layer="1"/>
+<wire x1="13.769" y1="33.457" x2="5.766" y2="25.454" width="5.5" layer="1"/>
+<wire x1="5.766" y1="25.454" x2="5.766" y2="16.243" width="5.5" layer="1"/>
+<wire x1="7.448" y1="14.561" x2="15.099" y2="14.561" width="5.5" layer="1"/>
+<wire x1="15.099" y1="14.561" x2="16.254" y2="15.716" width="5.5" layer="1"/>
+<wire x1="5.766" y1="16.243" x2="7.448" y2="14.561" width="5.5" layer="1"/>
+<wire x1="16.215" y1="33.457" x2="15.184" y2="33.457" width="4" layer="16"/>
+<wire x1="15.184" y1="33.457" x2="13.723" y2="33.457" width="5.5" layer="16"/>
+<wire x1="5.766" y1="25.5" x2="5.766" y2="16.289" width="5.5" layer="16"/>
+<wire x1="12.03719375" y1="14.561" x2="12.07519375" y2="14.599" width="5.5" layer="16"/>
+<wire x1="5.766" y1="16.289" x2="7.494" y2="14.561" width="5.5" layer="16"/>
+<wire x1="7.494" y1="14.561" x2="12.03719375" y2="14.561" width="5.5" layer="16"/>
+<wire x1="15.137" y1="14.599" x2="16.254" y2="15.716" width="5.5" layer="16"/>
+<wire x1="13.723" y1="33.457" x2="5.766" y2="25.5" width="5.5" layer="16"/>
+<wire x1="12.07519375" y1="14.599" x2="15.137" y2="14.599" width="5.5" layer="16"/>
+<wire x1="15.431" y1="33.436" x2="13.79" y2="33.436" width="0.1524" layer="1"/>
+<wire x1="13.79" y1="33.436" x2="13.769" y2="33.457" width="0.1524" layer="1"/>
 </signal>
 <signal name="2S_PROT">
-<contactref element="FUSE_HOLDER" pad="2_1"/>
-<contactref element="FUSE_HOLDER" pad="2_2"/>
 <contactref element="2S" pad="A"/>
 <contactref element="LEG0" pad="P$3"/>
@@
 <wire x1="28.338" y1="41.017" x2="28.431" y2="40.924" width="2" layer="1"/>
 <wire x1="34.3104" y1="25.5541" x2="35.3826" y2="26.6263" width="0.1524" layer="1"/>
-<wire x1="24.6606" y1="25.5541" x2="34.3104" y2="25.5541" width="0.1524" layer="1"/>
-<wire x1="23.9458" y1="26.2689" x2="24.6606" y2="25.5541" width="0.1524" layer="1"/>
+<wire x1="34.3104" y1="25.5541" x2="24.6606" y2="25.5541" width="0.1524" layer="1"/>
 <wire x1="35.3826" y1="26.6263" x2="35.4943" y2="26.7464" width="0.1524" layer="1"/>
-<wire x1="23.9458" y1="26.2689" x2="23.777" y2="26.274" width="0.1524" layer="1"/>
 <wire x1="36.8122" y1="3.9314" x2="31.9873" y2="8.7563" width="0.1524" layer="1"/>
 <wire x1="36.8122" y1="3.7527" x2="36.8122" y2="3.9314" width="0.1524" layer="1"/>
@@
 <wire x1="31.9873" y1="8.7563" x2="31.926" y2="8.888" width="0.1524" layer="1"/>
 <wire x1="38.5992" y1="12.3303" x2="38.591" y2="12.478" width="0.1524" layer="1"/>
+<contactref element="F1" pad="2_2"/>
+<contactref element="F1" pad="2_1"/>
+<wire x1="23.7197" y1="26.495" x2="22.558" y2="26.495" width="0.1524" layer="1"/>
+<wire x1="24.6606" y1="25.5541" x2="23.7197" y2="26.495" width="0.1524" layer="1"/>
 </signal>
 <signal name="2S_ESTOP">
-<contactref element="E_STOP" pad="+"/>
-<contactref element="FUSE_HOLDER" pad="1_2"/>
-<contactref element="FUSE_HOLDER" pad="1_1"/>
-<wire x1="15.5" y1="15.716" x2="21.635" y2="15.716" width="3" layer="16"/>
-<wire x1="21.635" y1="15.716" x2="23.777" y2="13.574" width="3" layer="16"/>
-<wire x1="23.777" y1="13.574" x2="23.777" y2="5.244" width="3" layer="16"/>
+<contactref element="F1" pad="1_2"/>
+<contactref element="F1" pad="1_1"/>
+<contactref element="E_STOP" pad="-"/>
+<wire x1="16.254" y1="8.516" x2="18.049" y2="8.516" width="5.5" layer="1"/>
+<wire x1="18.049" y1="8.516" x2="22.558" y2="13.025" width="5.5" layer="1"/>
+<wire x1="18.049" y1="8.516" x2="22.558" y2="13.025" width="5.5" layer="16"/>
+<wire x1="16.254" y1="8.516" x2="18.049" y2="8.516" width="5.5" layer="16"/>
+<wire x1="25.958" y1="13.025" x2="22.558" y2="13.025" width="5.5" layer="16"/>
+<wire x1="25.958" y1="13.025" x2="21.449" y2="8.516" width="5.5" layer="1"/>
+<wire x1="21.449" y1="8.516" x2="16.254" y2="8.516" width="5.5" layer="1"/>
 </signal>
 </signals>
